File: pcb/lolin-s2-uln2003a.kicad/lolin-s2-uln2003a.kicad_pcb (KiCad board)
At the start: 2 copper layers, 65.3 x 42.3 mm, 19 parts, among them J1 Conn_S2_Left, J10 Micro_SD_TF_PUSH, J11 Vin Barrel-Jack, J12 Conn_LED2, J2 Conn_S2_Right, J3 Conn_PWR, J4 Conn_Motor, J5 Conn_LED1, J6 Conn_LED3, J7 Conn_I2S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

Commit message: Rev. 2.00 of support-pcb
Parts:
- removed JP1: JMP_GAIN, Connector_PinHeader_2.54mm:PinHeader_1x03_P2.54mm_Vertical
- added C1: 100nF, Capacitor_SMD:C_0402_1005Metric, F.Cu at (87.5, 88.8)
- added J13: Conn_SUR2, Connector_JST:JST_SUR_BM02B-SURS-TF_1x02-1MP_P0.80mm_Vertical, F.Cu at (131.4, 105.9)
- added J14: Conn_SUR3, Connector_JST:JST_SUR_BM02B-SURS-TF_1x02-1MP_P0.80mm_Vertical, F.Cu at (131.3, 114.5)
- added J15: Conn_Neo, Connector_JST:JST_XH_B3B-XH-A_1x03_P2.50mm_Vertical, F.Cu at (78.8, 86.0)
- added J16: Conn_Extra, Connector_PinHeader_2.54mm:PinHeader_2x05_P2.54mm_Vertical, F.Cu at (105.7, 81.5)
- added R1: 33, Resistor_SMD:R_0402_1005Metric, F.Cu at (89.5, 86.8)
- added U2: DFR0299, user:DFR0299, F.Cu at (86.3, 108.4)
- added U3: 74LVC1G17, user:74LVC1G17GW_125, F.Cu at (89.8, 88.7)
- J10: value Micro_SD_TF_PUSH -> Conn_Spk; footprint user:TF-Push -> Connector_JST:JST_XH_B2B-XH-A_1x02_P2.50mm_Vertical
- J11: value Vin Barrel-Jack -> Conn_SUR1; footprint user:BarrelJack_CUI_PJ-102AH_Horizontal -> Connector_JST:JST_SUR_BM02B-SURS-TF_1x02-1MP_P0.80mm_Vertical
- J3: footprint Connector_PinHeader_2.54mm:PinHeader_1x04_P2.54mm_Vertical -> Connector_PinHeader_2.54mm:PinHeader_1x05_P2.54mm_Vertical
- J7: value Conn_I2S -> Conn_Player; footprint user:MAX98357A_Breakout -> Connector_JST:JST_XH_B2B-XH-A_1x02_P2.50mm_Vertical
- J8: footprint Connector_PinHeader_2.54mm:PinHeader_1x07_P2.54mm_Vertical -> Connector_PinHeader_2.54mm:PinHeader_1x06_P2.54mm_Vertical
- moved J10 16.6 mm to (78.9, 93.4)
- moved J3 15.0 mm to (126.0, 115.7), turned to 180 degrees
- moved U1 9.06 mm to (129.4, 84.2)
- moved J11 8.98 mm to (131.3, 97.5), turned to -90 degrees
- moved J7 7.66 mm to (87.5, 93.4), turned to 0 degrees
- moved J1 2.76 mm to (99.3, 92.9)
- moved J2 2.76 mm to (119.6, 92.9)
- moved J9 2.70 mm to (110.7, 110.3)
- moved H1 2.68 mm to (100.5, 79.8)
- moved H2 2.68 mm to (121.0, 79.8)
- moved H3 2.68 mm to (100.5, 116.1)
- moved H4 2.68 mm to (121.0, 116.1)
- moved REF** 2.63 mm to (98.1, 84.5)
Connections:
- J1 pad 12: /GPIO10 -> unconnected-(J1-Pin_12-Pad12)
- J10 pad 1: unconnected-(J10-DAT2-Pad1) -> Net-(J10-Pin_1)
- J10 pad 2: /GPIO4 -> Net-(J10-Pin_2)
- J11 pad 2: GND -> /LED1
- J2 pad 1: unconnected-(J2-Pin_1-Pad1) -> /GPIO40
- J2 pad 5: unconnected-(J2-Pin_5-Pad5) -> /GPIO36
- J3 pad 1: GND -> VBUS
- J3 pad 2: VBUS -> GND
- J3 pad 3: VCC -> VBUS
- J3 pad 4: GND -> VCC
- J7 pad 1: VBUS -> Net-(J7-Pin_1)
- J7 pad 2: GND -> Net-(J7-Pin_2)
Routing:
- net GND: track 47.4 -> 9.91 mm, vias 4 -> 1
- net VBUS: track 52.9 -> 16.0 mm
- net +3V3: track 24.2 -> 55.4 mm, vias 2 -> 0
- net Net-(J7-Pin_1): track 0.00 -> 27.1 mm
- net /GPIO36: track 0.00 -> 25.6 mm
- net Net-(J10-Pin_2): track 0.00 -> 25.6 mm
- net /GPIO10: track 21.9 -> 0.00 mm
- net Net-(J7-Pin_2): track 0.00 -> 20.9 mm
- net Net-(J10-Pin_1): track 0.00 -> 19.4 mm
- net /GPIO40: track 0.00 -> 16.5 mm
- net /GPIO8: track 19.8 -> 34.9 mm
- net /LED2: track 16.4 -> 31.4 mm, vias 0 -> 1
- net /LED1: track 10.4 -> 24.1 mm, vias 0 -> 1
- net /GPIO6: track 18.2 -> 30.2 mm
- net /LED3: track 24.3 -> 36.2 mm
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- added copper zone on F.Cu, net VBUS
- removed copper zone on F.Cu, net +3V3
Other:
- board text added: "+"
- board text added: "+-"
- board text added: "36 4"
- board text added: "38 6"
- board text added: "40 8"
- board text added: "9"
- board text added: "Blue"
- board text added: "DF-IO"
- board text added: "DF-Spk"
- board text added: "Motor"
- board text added: "Neopixel"
- board text added: "Offset L: 25.09"
- board text added: "Offset R: 19.73"
- board text added: "Orange"
- board text added: "Purple"
- board text added: "Rev. 2.00"
- board text added: "Yellow"
- board text added: "https://github.com/bablokb/christmas-pyramid"
- board text removed: "12dB"
- board text removed: "3V3"
- board text removed: "6dB"
- board text removed: "BCLK"
- board text removed: "DIN"
- board text removed: "GAIN"
- board text removed: "LRC"
- board text removed: "Rev. 1.01"
- board text removed: "SD"
- board text removed: "VIN"
- board text removed: "https://github.com/bablokb/motor-turntable"
- board text removed: "nc: 9dB"
